Commit message: Added gripper tool frame in urdf

File: lnt_urdf_description/urdf/lnt_urdf_description.urdf (robot description, URDF)
Before this commit: robot lnt_urdf_description, 9 links, 8 joints
Links:
- added link lnt_gripper_tool_frame, mass 0.0012; collision box size=0.01 0.01 0.01; visual box size=0.005 0.005 0.005
Joints:
- added joint lnt_gripper_tool_frame_joint: type fixed, parent link_6, child lnt_gripper_tool_frame, origin xyz=0 0 0.07 rpy=0 0 0

Commit message: Configured the tool frame in setup assistant.

File: lnt_urdf_description/urdf/lnt_urdf_description.urdf (robot description, URDF)
Before this commit: robot lnt_urdf_description, 10 links, 9 joints
Joints:
- joint lnt_gripper_tool_frame_joint: origin xyz=0 0 0.07 rpy=0 0 0 -> xyz=0 0 0.14 rpy=0 0 0

Commit message: Created new urdf with modified axes according to lnt requirement. Mande changes in initial theta calculation of end effector Added a local variable packet for processing the packet data correctly.

File: lnt_urdf_description/urdf/lnt_urdf_description.urdf (robot description, URDF)
Before this commit: robot lnt_urdf_description, 10 links, 9 joints
Links:
- link base_link: mass 0.854155845147982 -> 0.854155845147981
- link left_grip_link: mass 0.018543 -> 0.0185428410821073
- link link_2: mass 0.555909264188641 -> 0.555909264188642
- link link_5: mass 0.215222730814982 -> 0.215222730814981
- link link_6: mass 0.1106 -> 0.110597086440397
- link right_grip_link: mass 0.0185428410821074 -> 0.0185428410821077
Joints:
- joint joint1: origin xyz=0.039875 0.040125 0.3045 rpy=-3.0787E-17 1.1753E-16 1.5708 -> xyz=-0.04013 -0.04013 0.335 rpy=-6.163E-33 -3.3635E-16 5.5511E-17
- joint joint2: limit lower=-3.14 upper=0 effort=0 velocity=0 -> lower=0 upper=3.14 effort=0 velocity=0; origin xyz=0 0 0.0305 rpy=-1.5708 0 4.3305E-16 -> xyz=0 0 0 rpy=-1.5708 -8.4486E-17 4.6491E-16
- joint joint3: limit lower=0 upper=3.14159 effort=0 velocity=0 -> lower=-3.14 upper=0 effort=0 velocity=0; origin xyz=0.43132 -0.0012844 0 rpy=-2.3411E-15 -4.0406E-15 1.0617E-29 -> xyz=-0.43132 -0.0012844 0 rpy=2.9334E-15 -4.3854E-15 -1.3983E-29
- joint joint4: origin xyz=-0.2911 -0.05351 0 rpy=1.5708 2.6742E-15 -1.5708 -> xyz=0.2911 -0.05351 0 rpy=-1.5708 -3.8008E-15 -1.5708
- joint joint5: axis 0 0 1 -> 0 0 -1; origin xyz=0 0 0.041 rpy=1.5708 1.5708 0 -> xyz=0 0 0.041 rpy=1.5708 4.3758E-16 -3.0787E-17
- joint joint6: origin xyz=-0.122 0 0 rpy=1.5708 -1.1102E-16 -1.5708 -> xyz=0 0.122 0 rpy=-1.5708 3.0787E-17 2.7105E-16
- joint right_grip_joint: origin xyz=0.00038798 0.0423 0.1358 rpy=-1.5708 1.1403E-16 -3.1416 -> xyz=0.00038798 0.0423 0.1358 rpy=-1.5708 -1.108E-15 -3.1416
